Commit message: chore: Organize the URDF file
Align some physical parameters with the underlying layer.

File: nero/urdf/nero_description.urdf (robot description, URDF)
Before this commit: robot nero_description, 10 links, 9 joints
Links:
- removed link end_effector
- link base_link: mass 0.77 -> 1.06458435
- link link1: mass 0.77 -> 0.76710504; geometry collision mesh filename=package://agx_arm_description/agx_arm_urdf/nero/meshes/link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; visual mesh filename=package://agx_arm_description/agx_arm_urdf/nero/meshes/dae/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
- link link2: mass 0.49 -> 0.69381908; geometry collision mesh filename=package://agx_arm_description/agx_arm_urdf/nero/meshes/link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; visual mesh filename=package://agx_arm_description/agx_arm_urdf/nero/meshes/dae/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
- link link3: mass 0.67 -> 0.67246544; geometry collision mesh filename=package://agx_arm_description/agx_arm_urdf/nero/meshes/link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; visual mesh filename=package://agx_arm_description/agx_arm_urdf/nero/meshes/dae/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
- link link4: mass 0.41 -> 0.48451414; geometry collision mesh filename=package://agx_arm_description/agx_arm_urdf/nero/meshes/link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; visual mesh filename=package://agx_arm_description/agx_arm_urdf/nero/meshes/dae/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
- link link5: mass 0.56 -> 0.58368405; geometry collision mesh filename=package://agx_arm_description/agx_arm_urdf/nero/meshes/link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; visual mesh filename=package://agx_arm_description/agx_arm_urdf/nero/meshes/dae/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
- link link6: mass 0.31 -> 0.3140406; geometry collision mesh filename=package://agx_arm_description/agx_arm_urdf/nero/meshes/link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; visual mesh filename=package://agx_arm_description/agx_arm_urdf/nero/meshes/dae/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
- link link7: geometry collision mesh filename=package://agx_arm_description/agx_arm_urdf/nero/meshes/link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; visual mesh filename=package://agx_arm_description/agx_arm_urdf/nero/meshes/dae/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
Joints:
- removed joint end_effector_joint
- joint joint1: limit lower=-2.7 upper=2.7 effort=100 velocity=10 -> lower=-2.70526 upper=2.70526 effort=100 velocity=5
- joint joint2: limit lower=-1.74 upper=1.74 effort=100 velocity=10 -> lower=-1.74 upper=1.74 effort=100 velocity=5; origin xyz=0 0 0 rpy=1.5708 3.1415 0 -> xyz=0 0 0 rpy=1.5707963  3.1415926 0
- joint joint3: limit lower=-2.75 upper=2.75 effort=100 velocity=10 -> lower=-2.75 upper=2.75 effort=100 velocity=5; origin xyz=0 -0.31 0 rpy=-1.5708 0 3.1416 -> xyz=0 -0.31 0 rpy=-1.5707963  0 3.1415926926
- joint joint4: limit lower=-1.01 upper=2.14 effort=100 velocity=10 -> lower=-1.01 upper=2.14 effort=100 velocity=5; origin xyz=0 0 0 rpy=-1.5708 0 3.1416 -> xyz=0 0 0 rpy=-1.5707963  0 3.1415926926
- joint joint5: limit lower=-2.75 upper=2.75 effort=100 velocity=10 -> lower=-2.75 upper=2.75 effort=100 velocity=5; origin xyz=0 -0.27001 0 rpy=1.5708 -1.5708 0 -> xyz=0 -0.27001 0 rpy=1.5707963  -1.5707963  0
- joint joint6: limit lower=-0.73 upper=0.95 effort=100 velocity=10 -> lower=-0.73 upper=0.95 effort=100 velocity=5; origin xyz=0 0 0 rpy=1.5708 -1.5708 0 -> xyz=0 0 0 rpy=1.5707963  -1.5707963  0
- joint joint7: limit lower=-1.57 upper=1.57 effort=100 velocity=10 -> lower=-1.5707963 upper=1.5707963 effort=100 velocity=5; origin xyz=0 -0.0235 0 rpy=1.5708 0 0 -> xyz=0 -0.0235 0 rpy=1.5707963 0 0

File: piper/urdf/piper_description.urdf (robot description, URDF)
Before this commit: robot piper, 10 links, 9 joints
Links:
- removed link gripper_base
- removed link link7
- removed link link8
- added link world
- link base_link: geometry collision mesh filename=package://agx_arm_description/agx_arm_urdf/piper/meshes/bas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; visual mesh filename=package://agx_arm_description/agx_arm_urdf/piper/meshes/dae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
- link link1: geometry collision mesh filename=package://agx_arm_description/agx_arm_urdf/piper/meshes/lin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; visual mesh filename=package://agx_arm_description/agx_arm_urdf/piper/meshes/dae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
- link link2: geometry collision mesh filename=package://agx_arm_description/agx_arm_urdf/piper/meshes/lin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; visual mesh filename=package://agx_arm_description/agx_arm_urdf/piper/meshes/dae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
- link link3: geometry collision mesh filename=package://agx_arm_description/agx_arm_urdf/piper/meshes/lin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; visual mesh filename=package://agx_arm_description/agx_arm_urdf/piper/meshes/dae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
- link link4: geometry collision mesh filename=package://agx_arm_description/agx_arm_urdf/piper/meshes/lin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; visual mesh filename=package://agx_arm_description/agx_arm_urdf/piper/meshes/dae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
- link link5: geometry collision mesh filename=package://agx_arm_description/agx_arm_urdf/piper/meshes/lin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; visual mesh filename=package://agx_arm_description/agx_arm_urdf/piper/meshes/dae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
- link link6: geometry collision mesh filename=package://agx_arm_description/agx_arm_urdf/piper/meshes/lin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; visual mesh filename=package://agx_arm_description/agx_arm_urdf/piper/meshes/dae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
Joints:
- removed joint gripper_joint1
- removed joint gripper_joint2
- removed joint joint6_to_gripper_base
- added joint world_to_base_link: type fixed, parent world, child base_link, origin xyz=0 0 0 rpy=0 0 0
- joint joint1: limit lower=-2.618 upper=2.618 effort=100 velocity=5 -> lower=-2.6179938 upper=2.6179938 effort=100 velocity=5
- joint joint2: limit lower=0 upper=3.14 effort=100 velocity=5 -> lower=0 upper=3.1415926 effort=100 velocity=5; origin xyz=0 0 0 rpy=1.5708 -0.1359 -3.1416 -> xyz=0 0 0 rpy=1.5707963 -0.1357866 -3.1415926
- joint joint3: limit lower=-2.967 upper=0 effort=100 velocity=5 -> lower=-2.9670597 upper=0 effort=100 velocity=5; origin xyz=0.28503 0 0 rpy=0 0 -1.7939 -> xyz=0.28503 0 0 rpy=0 0 -1.7938494
- joint joint4: limit lower=-1.745 upper=1.745 effort=100 velocity=5 -> lower=-1.7453292 upper=1.7453292 effort=100 velocity=5; origin xyz=-0.021984 -0.25075 0 rpy=1.5708 0 0 -> xyz=-0.02198 -0.25075 0 rpy=1.5707963 0 0
- joint joint5: limit lower=-1.22 upper=1.22 effort=100 velocity=5 -> lower=-1.2217304 upper=1.2217304 effort=100 velocity=5; origin xyz=0 0 0 rpy=-1.5708 0 0 -> xyz=0 0 0 rpy=-1.5707963 0 0
- joint joint6: limit lower=-2.0944 upper=2.0944 effort=100 velocity=3 -> lower=-2.0943951 upper=2.0943951 effort=100 velocity=5; origin xyz=8.8259E-05 -0.091 0 rpy=1.5708 0 0 -> xyz=8.8259E-05 -0.091 0 rpy=1.5707963 0 0

File: piper_h/urdf/piper_h_description.urdf (robot description, URDF)
Before this commit: robot piper_h_description, 7 links, 6 joints
Links:
- added link world
- link base_link: mass 0.17076936349368 -> 1.02; geometry collision mesh filename=package://agx_arm_description/agx_arm_urdf/piper_h/meshes/b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; visual mesh filename=package://agx_arm_description/agx_arm_urdf/piper_h/meshes/d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
- link link1: mass 0.095130320813071 -> 0.71; geometry collision mesh filename=package://agx_arm_description/agx_arm_urdf/piper_h/meshes/l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; visual mesh filename=package://agx_arm_description/agx_arm_urdf/piper_h/meshes/d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
- link link2: mass 0.297349969020434 -> 1.16; geometry collision mesh filename=package://agx_arm_description/agx_arm_urdf/piper_h/meshes/l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; visual mesh filename=package://agx_arm_description/agx_arm_urdf/piper_h/meshes/d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
- link link3: mass 0.139005088174055 -> 0.5; geometry collision mesh filename=package://agx_arm_description/agx_arm_urdf/piper_h/meshes/l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; visual mesh filename=package://agx_arm_description/agx_arm_urdf/piper_h/meshes/d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
- link link4: mass 0.0625155037542606 -> 0.38; geometry collision mesh filename=package://agx_arm_description/agx_arm_urdf/piper_h/meshes/l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; visual mesh filename=package://agx_arm_description/agx_arm_urdf/piper_h/meshes/d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
- link link5: mass 0.0683301439531726 -> 0.39; geometry collision mesh filename=package://agx_arm_description/agx_arm_urdf/piper_h/meshes/l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; visual mesh filename=package://agx_arm_description/agx_arm_urdf/piper_h/meshes/d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
- link link6: mass 0.851169543242842 -> 0.007; geometry collision mesh filename=package://agx_arm_description/agx_arm_urdf/piper_h/meshes/l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; visual mesh filename=package://agx_arm_description/agx_arm_urdf/piper_h/meshes/d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
Joints:
- added joint world_to_base_link: type fixed, parent world, child base_link, origin xyz=0 0 0 rpy=0 0 0
- joint joint1: limit lower=-2.618 upper=2.618 effort=100 velocity=5 -> lower=-2.6179938 upper=2.6179938 effort=100 velocity=5
- joint joint2: limit lower=0 upper=3.14 effort=100 velocity=5 -> lower=0 upper=3.1415926 effort=100 velocity=5; origin xyz=0 0 0 rpy=1.5708 -0.13674 3.1416 -> xyz=0 0 0 rpy=1.5707963 -0.1357866 -3.1415926
- joint joint3: limit lower=-2.967 upper=0 effort=100 velocity=5 -> lower=-2.9670597 upper=0 effort=100 velocity=5; origin xyz=0.28508 0 0 rpy=0 0 -1.8796 -> xyz=0.28503 0 0 rpy=0 0 -1.7938494
- joint joint4: axis -0.087161 0 0.99619 -> 0 0 1; limit lower=-1.745 upper=1.745 effort=100 velocity=5 -> lower=-1.7453292 upper=1.7453292 effort=100 velocity=5; origin xyz=0 -0.25666 0 rpy=1.5708 0 0.17203 -> xyz=-0.02198 -0.25575 0 rpy=1.5707963 0 0
- joint joint5: limit lower=-1.22 upper=1.22 effort=100 velocity=5 -> lower=-1.2217304 upper=1.2217304 effort=100 velocity=5; origin xyz=0 0 0 rpy=-1.5708 -0.087272 0 -> xyz=0 0 0 rpy=-1.5707963 0 0
- joint joint6: axis -0.087161 0 0.99619 -> 0 0 1; limit lower=-2.0944 upper=2.0944 effort=100 velocity=3 -> lower=-2.0943951 upper=2.0943951 effort=100 velocity=5; origin xyz=0 -0.096 0 rpy=1.5708 0 0.087272 -> xyz=0 -0.0963 0 rpy=1.5707963 0 0

File: piper_l/urdf/piper_l_description.urdf (robot description, URDF)
Before this commit: robot piper_l_description, 7 links, 6 joints
Links:
- added link world
- link base_link: mass 0.228506683240186 -> 1.02; geometry collision mesh filename=package://agx_arm_description/agx_arm_urdf/piper_l/meshes/b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; visual mesh filename=package://agx_arm_description/agx_arm_urdf/piper_l/meshes/d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
- link link1: mass 0.104656591084326 -> 0.71; geometry collision mesh filename=package://agx_arm_description/agx_arm_urdf/piper_l/meshes/l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; visual mesh filename=package://agx_arm_description/agx_arm_urdf/piper_l/meshes/d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
- link link2: mass 0.289829779851577 -> 1.16; geometry collision mesh filename=package://agx_arm_description/agx_arm_urdf/piper_l/meshes/l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; visual mesh filename=package://agx_arm_description/agx_arm_urdf/piper_l/meshes/d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
- link link3: mass 0.144963320053385 -> 0.5; geometry collision mesh filename=package://agx_arm_description/agx_arm_urdf/piper_l/meshes/l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; visual mesh filename=package://agx_arm_description/agx_arm_urdf/piper_l/meshes/d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
- link link4: mass 0.063036548689954 -> 0.38; geometry collision mesh filename=package://agx_arm_description/agx_arm_urdf/piper_l/meshes/l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; visual mesh filename=package://agx_arm_description/agx_arm_urdf/piper_l/meshes/d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
- link link5: mass 0.069099989781007 -> 0.39; geometry collision mesh filename=package://agx_arm_description/agx_arm_urdf/piper_l/meshes/l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; visual mesh filename=package://agx_arm_description/agx_arm_urdf/piper_l/meshes/d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
- link link6: mass 0.00563228459599247 -> 0.007; geometry collision mesh filename=package://agx_arm_description/agx_arm_urdf/piper_l/meshes/l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; visual mesh filename=package://agx_arm_description/agx_arm_urdf/piper_l/meshes/d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
Joints:
- added joint world_to_base_link: type fixed, parent world, child base_link, origin xyz=0 0 0 rpy=0 0 0
- joint joint1: limit lower=-2.618 upper=2.618 effort=100 velocity=3 -> lower=-2.6179938 upper=2.6179938 effort=100 velocity=5
- joint joint2: limit lower=0 upper=3.14 effort=100 velocity=3 -> lower=0 upper=3.1415926 effort=100 velocity=5; origin xyz=0 0 0 rpy=1.5708 -0.1745 3.1416 -> xyz=0 0 0 rpy=1.5707963 -0.1357866 -3.1415926
- joint joint3: limit lower=-2.697 upper=0 effort=100 velocity=3 -> lower=-2.9670597 upper=0 effort=100 velocity=5; origin xyz=0.33823 0 0 rpy=0 0 -1.8325 -> xyz=0.33823 0 0 rpy=0 0 -1.7938494
- joint joint4: limit lower=-1.832 upper=1.832 effort=100 velocity=3 -> lower=-1.7453292 upper=1.7453292 effort=100 velocity=5; origin xyz=0 -0.3215 0 rpy=1.5708 0 0.1557 -> xyz=-0.02301 -0.32075 0 rpy=1.5707963 0 0
- joint joint5: axis 0 0 -1 -> 0 0 1; limit lower=-1.22 upper=1.22 effort=100 velocity=3 -> lower=-1.2217304 upper=1.2217304 effort=100 velocity=5; origin xyz=0 0 0 rpy=-1.5708 -0.087272 0 -> xyz=0 0 0 rpy=-1.5707963 0 0
- joint joint6: limit lower=-3.14 upper=3.14 effort=100 velocity=3 -> lower=-2.0943951 upper=2.0943951 effort=100 velocity=5; origin xyz=0 -0.091 0 rpy=1.5708 0 0 -> xyz=0 -0.091 0 rpy=1.5707963 0 0

File: piper_x/urdf/piper_x_description.urdf (robot description, URDF)
Before this commit: robot piper_x_description, 10 links, 9 joints
Links:
- removed link gripper_base
- removed link link7
- removed link link8
- added link world
- link base_link: mass 1.07 -> 1.02; geometry collision mesh filename=package://agx_arm_description/agx_arm_urdf/piper_x/meshes/b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; visual mesh filename=package://agx_arm_description/agx_arm_urdf/piper_x/meshes/d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
- link link1: geometry collision mesh filename=package://agx_arm_description/agx_arm_urdf/piper_x/meshes/l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; visual mesh filename=package://agx_arm_description/agx_arm_urdf/piper_x/meshes/d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
- link link2: geometry collision mesh filename=package://agx_arm_description/agx_arm_urdf/piper_x/meshes/l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; visual mesh filename=package://agx_arm_description/agx_arm_urdf/piper_x/meshes/d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
- link link3: geometry collision mesh filename=package://agx_arm_description/agx_arm_urdf/piper_x/meshes/l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; visual mesh filename=package://agx_arm_description/agx_arm_urdf/piper_x/meshes/d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
- link link4: mass 0.4 -> 0.39; geometry collision mesh filename=package://agx_arm_description/agx_arm_urdf/piper_x/meshes/l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; visual mesh filename=package://agx_arm_description/agx_arm_urdf/piper_x/meshes/d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
- link link5: geometry collision mesh filename=package://agx_arm_description/agx_arm_urdf/piper_x/meshes/l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; visual mesh filename=package://agx_arm_description/agx_arm_urdf/piper_x/meshes/d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
- link link6: geometry collision mesh filename=package://agx_arm_description/agx_arm_urdf/piper_x/meshes/l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; visual mesh filename=package://agx_arm_description/agx_arm_urdf/piper_x/meshes/d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
Joints:
- removed joint gripper_joint1
- removed joint gripper_joint2
- removed joint joint6_to_gripper_base
- added joint world_to_base_link: type fixed, parent world, child base_link, origin xyz=0 0 0 rpy=0 0 0
- joint joint1: limit lower=-2.618 upper=2.618 effort=100 velocity=10 -> lower=-2.6179938 upper=2.6179938 effort=100 velocity=5; origin xyz=0 0 0.123 rpy=0 0 0 -> xyz=0 0 0.123 rpy=0 0 3.1415926
- joint joint2: limit lower=0 upper=3.14 effort=100 velocity=10 -> lower=0 upper=3.1415926 effort=100 velocity=5; origin xyz=0 0 0 rpy=1.5708 -0.13586 3.1416 -> xyz=0 0 0 rpy=-1.5707963 -3.005806 -3.1415926
- joint joint3: limit lower=-2.9671 upper=0 effort=100 velocity=10 -> lower=-2.9670597 upper=0 effort=100 velocity=5; origin xyz=0.28503 0 0 rpy=0 0 2.8377 -> xyz=0.28503 0 0 rpy=0 0 2.8380798
- joint joint4: limit lower=-1.57 upper=1.57 effort=100 velocity=10 -> lower=-1.5707963 upper=1.5707963 effort=100 velocity=5; origin xyz=0.27264 0 0 rpy=0 0 0.075129 -> xyz=0.27364 0 0 rpy=0 0 0.0806342
- joint joint5: limit lower=-1.57 upper=1.57 effort=100 velocity=10 -> lower=-1.5707963 upper=1.5707963 effort=100 velocity=5; origin xyz=0.076857 0.00062395 0 rpy=-1.5708 0 0 -> xyz=0.07466 0 0 rpy=-1.5707963 1.5707963 0
- joint joint6: limit lower=-3.14 upper=3.14 effort=100 velocity=10 -> lower=-2.0943951 upper=2.0943951 effort=100 velocity=5; origin xyz=0.035 0 0 rpy=1.5708 0 1.5708 -> xyz=0 -0.035 0 rpy=1.5707963 0 0
