Commit message: chore: Add flange model

File: nero/urdf/nero_with_gripper_description.xacro (robot description, xacro)
@@ -23,5 +23,5 @@
         </collision>
     </link>
-    <joint name="gripper_base" type="fixed">
+    <joint name="gripper_base_joint" type="fixed">
         <origin xyz="0 0 0.0055" rpy="0 0 0"/>
         <parent link="gripper_flange"/>

File: nero/urdf/nero_with_gripper_flange_description.xacro (robot description, xacro)
@@ -23,5 +23,5 @@
         </collision>
     </link>
-    <joint name="gripper_flange" type="fixed">
+    <joint name="gripper_flange_joint" type="fixed">
         <origin xyz="0.032 0 -0.0235" rpy="-1.5708 0 -1.5708"/>
         <parent link="link7"/>

File: nero/urdf/nero_with_revo2_flange_description.xacro (robot description, xacro)
@@ -23,5 +23,5 @@
         </collision>
     </link>
-    <joint name="revo2_flange" type="fixed">
+    <joint name="revo2_flange_joint" type="fixed">
         <origin xyz="0.032 0 -0.0235" rpy="-1.5708 0 -1.5708"/>
         <parent link="link7"/>

File: piper/urdf/piper_with_gripper_description.xacro (robot description, xacro)
@@ -23,5 +23,5 @@
         </collision>
     </link>
-    <joint name="gripper_base" type="fixed">
+    <joint name="gripper_base_joint" type="fixed">
         <origin xyz="0 0 0" rpy="0 0 0"/>
         <parent link="link6"/>

File: piper/urdf/piper_with_left_revo2_description.xacro (robot description, xacro)
@@ -6,7 +6,31 @@
 <xacro:include filename="$(find agx_arm_description)/agx_arm_urdf/revo2/urdf/revo2_left_hand.urdf"/>
 <xacro:include filename="$(find agx_arm_description)/agx_arm_urdf/piper/urdf/piper_description.urdf"/>
+    <link name="flange_link">
+        <inertial>
+            <origin xyz="0.0 0.0 0.004" rpy="0 0 0"/>
+            <mass value="0.001"/>
+            <inertia ixx="0.00000001" ixy="0.00000000" ixz="0.00000000" iyy="0.00000001" iyz="0.00000000" izz="0.00000001"/>
+        </inertial>
+        <visual>
+            <origin xyz="0 0 0" rpy="0 0 0"/>
+            <geometry>
+                <mesh filename="package://agx_arm_description/agx_arm_urdf/piper/meshes/dae/flange.dae"/>
+            </geometry>
+        </visual>
+        <collision>
+            <origin xyz="0 0 0" rpy="0 0 0"/>
+            <geometry>
+                <mesh filename="package://agx_arm_description/agx_arm_urdf/piper/meshes/flange.stl"/>
+            </geometry>
+        </collision>
+    </link>
+    <joint name="flange_joint" type="fixed">
+        <origin xyz="0 0 0" rpy="0 0 0"/>
+        <parent link="link6"/>
+        <child link="flange_link"/>
+    </joint>
     <joint name="hand_base_joint" type="fixed">
-        <origin xyz="0.0 0.0 0.0" rpy="0 0 0"/>
-        <parent link="link6"/>
+        <origin xyz="0.0 0.0 0.008" rpy="0 0 0"/>
+        <parent link="flange_link"/>
         <child link="left_base_link"/>
         <axis xyz="0 0 0"/>

File: piper/urdf/piper_with_right_revo2_description.xacro (robot description, xacro)
@@ -6,7 +6,31 @@
 <xacro:include filename="$(find agx_arm_description)/agx_arm_urdf/revo2/urdf/revo2_right_hand.urdf"/>
 <xacro:include filename="$(find agx_arm_description)/agx_arm_urdf/piper/urdf/piper_description.urdf"/>
+    <link name="flange_link">
+        <inertial>
+            <origin xyz="0.0 0.0 0.004" rpy="0 0 0"/>
+            <mass value="0.001"/>
+            <inertia ixx="0.00000001" ixy="0.00000000" ixz="0.00000000" iyy="0.00000001" iyz="0.00000000" izz="0.00000001"/>
+        </inertial>
+        <visual>
+            <origin xyz="0 0 0" rpy="0 0 0"/>
+            <geometry>
+                <mesh filename="package://agx_arm_description/agx_arm_urdf/piper/meshes/dae/flange.dae"/>
+            </geometry>
+        </visual>
+        <collision>
+            <origin xyz="0 0 0" rpy="0 0 0"/>
+            <geometry>
+                <mesh filename="package://agx_arm_description/agx_arm_urdf/piper/meshes/flange.stl"/>
+            </geometry>
+        </collision>
+    </link>
+    <joint name="flange_joint" type="fixed">
+        <origin xyz="0 0 0" rpy="0 0 0"/>
+        <parent link="link6"/>
+        <child link="flange_link"/>
+    </joint>
     <joint name="hand_base_joint" type="fixed">
-        <origin xyz="0.0 0.0 0.0" rpy="0 0 0"/>
-        <parent link="link6"/>
+        <origin xyz="0.0 0.0 0.008" rpy="0 0 0"/>
+        <parent link="flange_link"/>
         <child link="right_base_link"/>
         <axis xyz="0 0 0"/>

File: piper_h/urdf/piper_h_with_gripper_description.xacro (robot description, xacro)
@@ -23,5 +23,5 @@
         </collision>
     </link>
-    <joint name="gripper_base" type="fixed">
+    <joint name="gripper_base_joint" type="fixed">
         <origin xyz="0 0 0" rpy="0 0 0"/>
         <parent link="link6"/>

File: piper_h/urdf/piper_h_with_left_revo2_description.xacro (robot description, xacro)
@@ -6,7 +6,31 @@
 <xacro:include filename="$(find agx_arm_description)/agx_arm_urdf/revo2/urdf/revo2_left_hand.urdf"/>
 <xacro:include filename="$(find agx_arm_description)/agx_arm_urdf/piper_h/urdf/piper_h_description.urdf"/>
+    <link name="flange_link">
+        <inertial>
+            <origin xyz="0.0 0.0 0.004" rpy="0 0 0"/>
+            <mass value="0.001"/>
+            <inertia ixx="0.00000001" ixy="0.00000000" ixz="0.00000000" iyy="0.00000001" iyz="0.00000000" izz="0.00000001"/>
+        </inertial>
+        <visual>
+            <origin xyz="0 0 0" rpy="0 0 0"/>
+            <geometry>
+                <mesh filename="package://agx_arm_description/agx_arm_urdf/piper_h/meshes/dae/flange.dae"/>
+            </geometry>
+        </visual>
+        <collision>
+            <origin xyz="0 0 0" rpy="0 0 0"/>
+            <geometry>
+                <mesh filename="package://agx_arm_description/agx_arm_urdf/piper_h/meshes/flange.stl"/>
+            </geometry>
+        </collision>
+    </link>
+    <joint name="flange_joint" type="fixed">
+        <origin xyz="0 0 0" rpy="0 0 0"/>
+        <parent link="link6"/>
+        <child link="flange_link"/>
+    </joint>
     <joint name="hand_base_joint" type="fixed">
-        <origin xyz="0.0 0.0 0.0" rpy="0 0 0"/>
-        <parent link="link6"/>
+        <origin xyz="0.0 0.0 0.008" rpy="0 0 0"/>
+        <parent link="flange_link"/>
         <child link="left_base_link"/>
         <axis xyz="0 0 0"/>

File: piper_h/urdf/piper_h_with_right_revo2_description.xacro (robot description, xacro)
@@ -6,7 +6,31 @@
 <xacro:include filename="$(find agx_arm_description)/agx_arm_urdf/revo2/urdf/revo2_right_hand.urdf"/>
 <xacro:include filename="$(find agx_arm_description)/agx_arm_urdf/piper_h/urdf/piper_h_description.urdf"/>
+    <link name="flange_link">
+        <inertial>
+            <origin xyz="0.0 0.0 0.004" rpy="0 0 0"/>
+            <mass value="0.001"/>
+            <inertia ixx="0.00000001" ixy="0.00000000" ixz="0.00000000" iyy="0.00000001" iyz="0.00000000" izz="0.00000001"/>
+        </inertial>
+        <visual>
+            <origin xyz="0 0 0" rpy="0 0 0"/>
+            <geometry>
+                <mesh filename="package://agx_arm_description/agx_arm_urdf/piper_h/meshes/dae/flange.dae"/>
+            </geometry>
+        </visual>
+        <collision>
+            <origin xyz="0 0 0" rpy="0 0 0"/>
+            <geometry>
+                <mesh filename="package://agx_arm_description/agx_arm_urdf/piper_h/meshes/flange.stl"/>
+            </geometry>
+        </collision>
+    </link>
+    <joint name="flange_joint" type="fixed">
+        <origin xyz="0 0 0" rpy="0 0 0"/>
+        <parent link="link6"/>
+        <child link="flange_link"/>
+    </joint>
     <joint name="hand_base_joint" type="fixed">
-        <origin xyz="0.0 0.0 0.0" rpy="0 0 0"/>
-        <parent link="link6"/>
+        <origin xyz="0.0 0.0 0.008" rpy="0 0 0"/>
+        <parent link="flange_link"/>
         <child link="right_base_link"/>
         <axis xyz="0 0 0"/>

File: piper_l/urdf/piper_l_with_gripper_description.xacro (robot description, xacro)
@@ -23,5 +23,5 @@
         </collision>
     </link>
-    <joint name="gripper_base" type="fixed">
+    <joint name="gripper_base_joint" type="fixed">
         <origin xyz="0 0 0" rpy="0 0 0"/>
         <parent link="link6"/>

File: piper_l/urdf/piper_l_with_left_revo2_description.xacro (robot description, xacro)
@@ -6,7 +6,31 @@
 <xacro:include filename="$(find agx_arm_description)/agx_arm_urdf/revo2/urdf/revo2_left_hand.urdf"/>
 <xacro:include filename="$(find agx_arm_description)/agx_arm_urdf/piper_l/urdf/piper_l_description.urdf"/>
+    <link name="flange_link">
+        <inertial>
+            <origin xyz="0.0 0.0 0.004" rpy="0 0 0"/>
+            <mass value="0.001"/>
+            <inertia ixx="0.00000001" ixy="0.00000000" ixz="0.00000000" iyy="0.00000001" iyz="0.00000000" izz="0.00000001"/>
+        </inertial>
+        <visual>
+            <origin xyz="0 0 0" rpy="0 0 0"/>
+            <geometry>
+                <mesh filename="package://agx_arm_description/agx_arm_urdf/piper_l/meshes/dae/flange.dae"/>
+            </geometry>
+        </visual>
+        <collision>
+            <origin xyz="0 0 0" rpy="0 0 0"/>
+            <geometry>
+                <mesh filename="package://agx_arm_description/agx_arm_urdf/piper_l/meshes/flange.stl"/>
+            </geometry>
+        </collision>
+    </link>
+    <joint name="flange_joint" type="fixed">
+        <origin xyz="0 0 0" rpy="0 0 0"/>
+        <parent link="link6"/>
+        <child link="flange_link"/>
+    </joint>
     <joint name="hand_base_joint" type="fixed">
-        <origin xyz="0.0 0.0 0.0" rpy="0 0 0"/>
-        <parent link="link6"/>
+        <origin xyz="0.0 0.0 0.008" rpy="0 0 0"/>
+        <parent link="flange_link"/>
         <child link="left_base_link"/>
         <axis xyz="0 0 0"/>

File: piper_l/urdf/piper_l_with_right_revo2_description.xacro (robot description, xacro)
@@ -6,7 +6,31 @@
 <xacro:include filename="$(find agx_arm_description)/agx_arm_urdf/revo2/urdf/revo2_right_hand.urdf"/>
 <xacro:include filename="$(find agx_arm_description)/agx_arm_urdf/piper_l/urdf/piper_l_description.urdf"/>
+    <link name="flange_link">
+        <inertial>
+            <origin xyz="0.0 0.0 0.004" rpy="0 0 0"/>
+            <mass value="0.001"/>
+            <inertia ixx="0.00000001" ixy="0.00000000" ixz="0.00000000" iyy="0.00000001" iyz="0.00000000" izz="0.00000001"/>
+        </inertial>
+        <visual>
+            <origin xyz="0 0 0" rpy="0 0 0"/>
+            <geometry>
+                <mesh filename="package://agx_arm_description/agx_arm_urdf/piper_l/meshes/dae/flange.dae"/>
+            </geometry>
+        </visual>
+        <collision>
+            <origin xyz="0 0 0" rpy="0 0 0"/>
+            <geometry>
+                <mesh filename="package://agx_arm_description/agx_arm_urdf/piper_l/meshes/flange.stl"/>
+            </geometry>
+        </collision>
+    </link>
+    <joint name="flange_joint" type="fixed">
+        <origin xyz="0 0 0" rpy="0 0 0"/>
+        <parent link="link6"/>
+        <child link="flange_link"/>
+    </joint>
     <joint name="hand_base_joint" type="fixed">
-        <origin xyz="0.0 0.0 0.0" rpy="0 0 0"/>
-        <parent link="link6"/>
+        <origin xyz="0.0 0.0 0.008" rpy="0 0 0"/>
+        <parent link="flange_link"/>
         <child link="right_base_link"/>
         <axis xyz="0 0 0"/>

File: piper_x/urdf/piper_x_with_gripper_description.xacro (robot description, xacro)
@@ -23,5 +23,5 @@
         </collision>
     </link>
-    <joint name="gripper_base" type="fixed">
+    <joint name="gripper_base_joint" type="fixed">
         <origin xyz="0 0 0" rpy="0 0 1.5707963"/>
         <parent link="link6"/>

File: piper_x/urdf/piper_x_with_left_revo2_description.xacro (robot description, xacro)
@@ -6,7 +6,31 @@
 <xacro:include filename="$(find agx_arm_description)/agx_arm_urdf/revo2/urdf/revo2_left_hand.urdf"/>
 <xacro:include filename="$(find agx_arm_description)/agx_arm_urdf/piper_x/urdf/piper_x_description.urdf"/>
+    <link name="flange_link">
+        <inertial>
+            <origin xyz="0.0 0.0 0.004" rpy="0 0 0"/>
+            <mass value="0.001"/>
+            <inertia ixx="0.00000001" ixy="0.00000000" ixz="0.00000000" iyy="0.00000001" iyz="0.00000000" izz="0.00000001"/>
+        </inertial>
+        <visual>
+            <origin xyz="0 0 0" rpy="0 0 0"/>
+            <geometry>
+                <mesh filename="package://agx_arm_description/agx_arm_urdf/piper_x/meshes/dae/flange.dae"/>
+            </geometry>
+        </visual>
+        <collision>
+            <origin xyz="0 0 0" rpy="0 0 0"/>
+            <geometry>
+                <mesh filename="package://agx_arm_description/agx_arm_urdf/piper_x/meshes/flange.stl"/>
+            </geometry>
+        </collision>
+    </link>
+    <joint name="flange_joint" type="fixed">
+        <origin xyz="0 0 0" rpy="0 0 1.5707963"/>
+        <parent link="link6"/>
+        <child link="flange_link"/>
+    </joint>
     <joint name="hand_base_joint" type="fixed">
-        <origin xyz="0.0 0.0 0.0" rpy="0 0 1.5707963"/>
-        <parent link="link6"/>
+        <origin xyz="0.0 0.0 0.008" rpy="0 0 0"/>
+        <parent link="flange_link"/>
         <child link="left_base_link"/>
         <axis xyz="0 0 0"/>

File: piper_x/urdf/piper_x_with_right_revo2_description.xacro (robot description, xacro)
@@ -6,7 +6,31 @@
 <xacro:include filename="$(find agx_arm_description)/agx_arm_urdf/revo2/urdf/revo2_right_hand.urdf"/>
 <xacro:include filename="$(find agx_arm_description)/agx_arm_urdf/piper_x/urdf/piper_x_description.urdf"/>
+    <link name="flange_link">
+        <inertial>
+            <origin xyz="0.0 0.0 0.004" rpy="0 0 0"/>
+            <mass value="0.001"/>
+            <inertia ixx="0.00000001" ixy="0.00000000" ixz="0.00000000" iyy="0.00000001" iyz="0.00000000" izz="0.00000001"/>
+        </inertial>
+        <visual>
+            <origin xyz="0 0 0" rpy="0 0 0"/>
+            <geometry>
+                <mesh filename="package://agx_arm_description/agx_arm_urdf/piper_x/meshes/dae/flange.dae"/>
+            </geometry>
+        </visual>
+        <collision>
+            <origin xyz="0 0 0" rpy="0 0 0"/>
+            <geometry>
+                <mesh filename="package://agx_arm_description/agx_arm_urdf/piper_x/meshes/flange.stl"/>
+            </geometry>
+        </collision>
+    </link>
+    <joint name="flange_joint" type="fixed">
+        <origin xyz="0 0 0" rpy="0 0 1.5707963"/>
+        <parent link="link6"/>
+        <child link="flange_link"/>
+    </joint>
     <joint name="hand_base_joint" type="fixed">
-        <origin xyz="0.0 0.0 0.0" rpy="0 0 1.5707963"/>
-        <parent link="link6"/>
+        <origin xyz="0.0 0.0 0.008" rpy="0 0 0"/>
+        <parent link="flange_link"/>
         <child link="right_base_link"/>
         <axis xyz="0 0 0"/>
